File: BufferedDifferenceAmplifierId.sch (KiCad schematic (older format))
At the start: 13 parts, among them U1 LMC6044, U2 LMC6044, U3 LM324

Commit message: Added negative swing on gate-source bias and RTD connection.
Parts:
- R40, R42, R44, R45, R46, R47, R48, R49: value 100k -> 10k
Changed lines of the file:
@@
 AR Path="/5F4F2130/5F4B27DF" Ref="R?"  Part="1"
 F 0 "R40" H 5400 2700 50  0000 R CNN
-F 1 "100k" H 5400 2800 50  0000 R CNN
+F 1 "10k" H 5400 2800 50  0000 R CNN
 F 2 "Resistor_SMD:R_0603_1608Metric" V 5080 2750 50  0001 C CNN
 F 3 "~" H 5150 2750 50  0001 C CNN
@@
 AR Path="/5F4F2130/5F4F2F18" Ref="R?"  Part="1"
 F 0 "R44" V 5500 3400 50  0000 C CNN
-F 1 "100k" V 5400 3350 50  0000 C CNN
+F 1 "10k" V 5400 3350 50  0000 C CNN
 F 2 "Resistor_SMD:R_0603_1608Metric" V 5530 3350 50  0001 C CNN
 F 3 "~" H 5600 3350 50  0001 C CNN
@@
 AR Path="/5F4F2130/5F4B87BB" Ref="R?"  Part="1"
 F 0 "R46" V 6400 3350 50  0000 C CNN
-F 1 "100k" V 6316 3350 50  0000 C CNN
+F 1 "10k" V 6316 3350 50  0000 C CNN
 F 2 "Resistor_SMD:R_0603_1608Metric" V 6130 3350 50  0001 C CNN
 F 3 "~" H 6200 3350 50  0001 C CNN
@@
 AR Path="/5F4F2130/5F4F5397" Ref="R?"  Part="1"
 F 0 "R42" H 5400 4000 50  0000 R CNN
-F 1 "100k" H 5400 4100 50  0000 R CNN
+F 1 "10k" H 5400 4100 50  0000 R CNN
 F 2 "Resistor_SMD:R_0603_1608Metric" V 5080 4050 50  0001 C CNN
 F 3 "~" H 5150 4050 50  0001 C CNN
@@
 AR Path="/5F4F2130/5F4F2F1C" Ref="R?"  Part="1"
 F 0 "R47" V 6300 3550 50  0000 C CNN
-F 1 "100k" V 6400 3550 50  0000 C CNN
+F 1 "10k" V 6400 3550 50  0000 C CNN
 F 2 "Resistor_SMD:R_0603_1608Metric" V 6130 3550 50  0001 C CNN
 F 3 "~" H 6200 3550 50  0001 C CNN
@@
 AR Path="/5F4F2130/5F4F2F1D" Ref="R?"  Part="1"
 F 0 "R49" V 7050 3750 50  0000 C CNN
-F 1 "100k" V 7150 3750 50  0000 C CNN
+F 1 "10k" V 7150 3750 50  0000 C CNN
 F 2 "Resistor_SMD:R_0603_1608Metric" V 6880 3750 50  0001 C CNN
 F 3 "~" H 6950 3750 50  0001 C CNN
@@
 AR Path="/5F4F2130/5F4F2F1E" Ref="R?"  Part="1"
 F 0 "R48" H 6550 2800 50  0000 R CNN
-F 1 "100k" H 6600 2900 50  0000 R CNN
+F 1 "10k" H 6600 2900 50  0000 R CNN
 F 2 "Resistor_SMD:R_0603_1608Metric" V 6430 3150 50  0001 C CNN
 F 3 "~" H 6500 3150 50  0001 C CNN
@@
 AR Path="/5F4F2130/5F4F2F1F" Ref="R?"  Part="1"
 F 0 "R45" V 5700 4650 50  0000 C CNN
-F 1 "100k" V 5800 4650 50  0000 C CNN
+F 1 "10k" V 5800 4650 50  0000 C CNN
 F 2 "Resistor_SMD:R_0603_1608Metric" V 5530 4650 50  0001 C CNN
 F 3 "~" H 5600 4650 50  0001 C CNN
