File: BufferedDifferenceAmplifierIg.sch (KiCad schematic (older format))
At the start: 13 parts, among them U1 LMC6044, U2 LMC6044, U3 LM324

Commit message: Added negative swing on gate-source bias and RTD connection.
Parts:
- R30, R32, R34, R35, R36, R37, R38, R39: value 100k -> 10k
Changed lines of the file:
@@
 AR Path="/5F4F2130/5F4F538F" Ref="R30"  Part="1"
 F 0 "R30" H 5400 2700 50  0000 R CNN
-F 1 "100k" H 5400 2800 50  0000 R CNN
+F 1 "10k" H 5400 2800 50  0000 R CNN
 F 2 "Resistor_SMD:R_0603_1608Metric" V 5080 2750 50  0001 C CNN
 F 3 "~" H 5150 2750 50  0001 C CNN
@@
 AR Path="/5F4F2130/5F4B7256" Ref="R34"  Part="1"
 F 0 "R34" V 5500 3400 50  0000 C CNN
-F 1 "100k" V 5400 3350 50  0000 C CNN
+F 1 "10k" V 5400 3350 50  0000 C CNN
 F 2 "Resistor_SMD:R_0603_1608Metric" V 5530 3350 50  0001 C CNN
 F 3 "~" H 5600 3350 50  0001 C CNN
@@
 AR Path="/5F4F2130/5F4F5395" Ref="R36"  Part="1"
 F 0 "R36" V 6400 3350 50  0000 C CNN
-F 1 "100k" V 6316 3350 50  0000 C CNN
+F 1 "10k" V 6316 3350 50  0000 C CNN
 F 2 "Resistor_SMD:R_0603_1608Metric" V 6130 3350 50  0001 C CNN
 F 3 "~" H 6200 3350 50  0001 C CNN
@@
 AR Path="/5F4F2130/5F4B9E0F" Ref="R32"  Part="1"
 F 0 "R32" H 5400 4000 50  0000 R CNN
-F 1 "100k" H 5400 4100 50  0000 R CNN
+F 1 "10k" H 5400 4100 50  0000 R CNN
 F 2 "Resistor_SMD:R_0603_1608Metric" V 5080 4050 50  0001 C CNN
 F 3 "~" H 5150 4050 50  0001 C CNN
@@
 AR Path="/5F4F2130/5F4F5398" Ref="R37"  Part="1"
 F 0 "R37" V 6300 3550 50  0000 C CNN
-F 1 "100k" V 6400 3550 50  0000 C CNN
+F 1 "10k" V 6400 3550 50  0000 C CNN
 F 2 "Resistor_SMD:R_0603_1608Metric" V 6130 3550 50  0001 C CNN
 F 3 "~" H 6200 3550 50  0001 C CNN
@@
 AR Path="/5F4F2130/5F4F5399" Ref="R39"  Part="1"
 F 0 "R39" V 7050 3750 50  0000 C CNN
-F 1 "100k" V 7150 3750 50  0000 C CNN
+F 1 "10k" V 7150 3750 50  0000 C CNN
 F 2 "Resistor_SMD:R_0603_1608Metric" V 6880 3750 50  0001 C CNN
 F 3 "~" H 6950 3750 50  0001 C CNN
@@
 AR Path="/5F4F2130/5F4F539A" Ref="R38"  Part="1"
 F 0 "R38" H 6550 2800 50  0000 R CNN
-F 1 "100k" H 6600 2900 50  0000 R CNN
+F 1 "10k" H 6600 2900 50  0000 R CNN
 F 2 "Resistor_SMD:R_0603_1608Metric" V 6430 3150 50  0001 C CNN
 F 3 "~" H 6500 3150 50  0001 C CNN
@@
 AR Path="/5F4F2130/5F4F539B" Ref="R35"  Part="1"
 F 0 "R35" V 5700 4650 50  0000 C CNN
-F 1 "100k" V 5800 4650 50  0000 C CNN
+F 1 "10k" V 5800 4650 50  0000 C CNN
 F 2 "Resistor_SMD:R_0603_1608Metric" V 5530 4650 50  0001 C CNN
 F 3 "~" H 5600 4650 50  0001 C CNN
