File: BufferedDifferenceAmplifierVg.sch (KiCad schematic (older format))
At the start: 13 parts, among them U1 LMC6044, U2 LMC6044, U3 LM324

Commit message: Added negative swing on gate-source bias and RTD connection.
Connections:
- net GND: no longer R28.2
- new net +5V: R28.2
Changed lines of the file:
@@
 	6500 3000 6500 2950
-Wire Wire Line
-	6500 2950 6650 2950
-Wire Wire Line
-	6650 2950 6650 3000
 Wire Wire Line
 	6500 3300 6500 3350
@@
 $Comp
 L power:GND #PWR?
-U 1 1 5F4F2122
-P 6650 3000
-AR Path="/5F4838F1/5F4F2122" Ref="#PWR?"  Part="1"
-AR Path="/5F4BF3F3/5F4F2122" Ref="#PWR?"  Part="1"
-AR Path="/5F4C15ED/5F4F2122" Ref="#PWR?"  Part="1"
-AR Path="/5F4EF06B/5F4F2122" Ref="#PWR031"  Part="1"
-AR Path="/5F4F133C/5F4F2122" Ref="#PWR?"  Part="1"
-F 0 "#PWR031" H 6650 2750 50  0001 C CNN
-F 1 "GND" H 6655 2827 50  0000 C CNN
-F 2 "" H 6650 3000 50  0001 C CNN
-F 3 "" H 6650 3000 50  0001 C CNN
-	1    6650 3000
-	1    0    0    -1
-$EndComp
-$Comp
-L power:GND #PWR?
 U 1 1 5F4F2123
 P 5150 4700
@@
 AR Path="/5F4EF06B/5F4BB3A7" Ref="R28"  Part="1"
 AR Path="/5F4F133C/5F4BB3A7" Ref="R?"  Part="1"
-F 0 "R28" H 6550 2800 50  0000 R CNN
-F 1 "100k" H 6600 2900 50  0000 R CNN
+F 0 "R28" H 6400 3050 50  0000 R CNN
+F 1 "100k" H 6400 3150 50  0000 R CNN
 F 2 "Resistor_SMD:R_0603_1608Metric" V 6430 3150 50  0001 C CNN
 F 3 "~" H 6500 3150 50  0001 C CNN
@@
 	0    1    1    0
 $EndComp
+$Comp
+L power:+5V #PWR0114
+U 1 1 5F4C8B21
+P 6500 2950
+F 0 "#PWR0114" H 6500 2800 50  0001 C CNN
+F 1 "+5V" H 6515 3123 50  0000 C CNN
+F 2 "" H 6500 2950 50  0001 C CNN
+F 3 "" H 6500 2950 50  0001 C CNN
+	1    6500 2950
+	1    0    0    -1
+$EndComp
 $EndSCHEMATC
